File: hardware/Windig_Kicad.sch (KiCad schematic (older format))
At the start: 31 parts, among them J1 Barrel_Jack, J10 USB_B, J11 Conn_02x03, J2 Conn_01x04, J3 Conn_01x04, J4 Conn_01x04, J5 Conn_01x04, J6 Conn_01x04, J7 Conn_01x04, J8 Conn_01x04, J9 Conn_01x04, SW1 SW_SPDT, SW2 SW_SPDT, U1 ATmega328P-PU, X1 16Mhz

Commit message: Rough component placemunt update
Parts:
- removed TP1: RESET, Connector_PinHeader_2.54mm:PinHeader_1x01_P2.54mm_Vertical, symbol 4ms-headers:Test_Point
- added H1, H2, H3, H4: MountingHole, MountingHole:MountingHole_3.2mm_M3, symbol Mechanical:MountingHole
- C5: footprint Capacitor_THT:C_Disc_D6.0mm_W4.4mm_P5.00mm -> Capacitor_THT:C_Disc_D3.8mm_W2.6mm_P2.50mm
- R2, R3, R4, R5, R6, R7: footprint Resistor_THT:R_Axial_DIN0207_L6.3mm_D2.5mm_P7.62mm_Horizontal -> Resistor_THT:R_Axial_DIN0309_L9.0mm_D3.2mm_P2.54mm_Vertical
- U1: symbol MCU_Microchip_ATmega:ATmega328P-PU -> Windig_Kicad-rescue:ATmega328P-PU-MCU_Microchip_ATmega
Connections:
- net 5v: no longer U1.21 (AREF)
- net TACH1A: now also U1.24 (PC1); no longer U1.23 (PC0)
- net TACH1B: now also U1.23 (PC0); no longer U1.24 (PC1)
Changed lines of the file:
@@
 EESchema Schematic File Version 4
-LIBS:Windig_Kicad-cache
 EELAYER 30 0
 EELAYER END
@@
 F 0 "R6" V 6350 6000 50  0000 C CNN
 F 1 "1k5" V 6350 5800 50  0000 C CNN
-F 2 "Resistor_THT:R_Axial_DIN0207_L6.3mm_D2.5mm_P7.62mm_Horizontal" V 6380 5900 50  0001 C CNN
+F 2 "Resistor_THT:R_Axial_DIN0309_L9.0mm_D3.2mm_P2.54mm_Vertical" V 6380 5900 50  0001 C CNN
 F 3 "" H 6450 5900 50  0001 C CNN
 	1    6450 5900
@@
 MISO
 $Comp
-L MCU_Microchip_ATmega:ATmega328P-PU U1
+L Windig_Kicad-rescue:ATmega328P-PU-MCU_Microchip_ATmega U1
 U 1 1 5DFC356B
 P 2250 5000
@@
 $EndComp
 Wire Wire Line
-	4100 2350 4000 2350
-Wire Wire Line
 	3600 2350 3400 2350
-Wire Wire Line
-	4000 2350 4000 2450
-Connection ~ 4000 2350
-Wire Wire Line
-	4000 2350 3900 2350
 $Comp
 L 4ms-power:GND #PWR015
@@
 F 0 "R5" V 6350 5700 50  0000 C CNN
 F 1 "62r" V 6350 5500 50  0000 C CNN
-F 2 "Resistor_THT:R_Axial_DIN0207_L6.3mm_D2.5mm_P7.62mm_Horizontal" V 6380 5600 50  0001 C CNN
+F 2 "Resistor_THT:R_Axial_DIN0309_L9.0mm_D3.2mm_P2.54mm_Vertical" V 6380 5600 50  0001 C CNN
 F 3 "" H 6450 5600 50  0001 C CNN
 	1    6450 5600
@@
 F 0 "R4" V 6350 5200 50  0000 C CNN
 F 1 "62r" V 6350 5000 50  0000 C CNN
-F 2 "Resistor_THT:R_Axial_DIN0207_L6.3mm_D2.5mm_P7.62mm_Horizontal" V 6380 5100 50  0001 C CNN
+F 2 "Resistor_THT:R_Axial_DIN0309_L9.0mm_D3.2mm_P2.54mm_Vertical" V 6380 5100 50  0001 C CNN
 F 3 "" H 6450 5100 50  0001 C CNN
 	1    6450 5100
@@
 F 0 "R3" H 6650 4850 50  0000 C CNN
 F 1 "1k" H 6650 4700 50  0000 C CNN
-F 2 "Resistor_THT:R_Axial_DIN0207_L6.3mm_D2.5mm_P7.62mm_Horizontal" V 6680 4750 50  0001 C CNN
+F 2 "Resistor_THT:R_Axial_DIN0309_L9.0mm_D3.2mm_P2.54mm_Vertical" V 6680 4750 50  0001 C CNN
 F 3 "" H 6750 4750 50  0001 C CNN
 	1    6750 4750
@@
 F 0 "C5" H 6265 4546 50  0000 L CNN
 F 1 "100nF" H 6265 4455 50  0000 L CNN
-F 2 "Capacitor_THT:C_Disc_D6.0mm_W4.4mm_P5.00mm" H 6188 4350 50  0001 C CNN
+F 2 "Capacitor_THT:C_Disc_D3.8mm_W2.6mm_P2.50mm" H 6188 4350 50  0001 C CNN
 F 3 "" H 6150 4500 50  0001 C CNN
 	1    6150 4500
@@
 Text GLabel 3350 5800 2    50   Input ~ 0
 PWM1
+Text GLabel 3350 4800 2    50   Input ~ 0
+TACH1A
 Text GLabel 3350 4700 2    50   Input ~ 0
-TACH1A
-Text GLabel 3350 4800 2    50   Input ~ 0
 TACH1B
 Text GLabel 3350 4000 2    50   Input ~ 0
@@
 	2400 850  3050 850
 Wire Wire Line
-	1650 3800 1500 3800
-Wire Wire Line
-	1500 3800 1500 3350
-Wire Wire Line
-	1500 3350 2250 3350
-Wire Wire Line
-	1300 3350 1500 3350
-Connection ~ 1500 3350
-Wire Wire Line
 	3050 1300 3050 1400
 Connection ~ 3050 850
@@
 Wire Wire Line
 	3050 1400 3050 1550
-$Comp
-L 4ms-headers:Test_Point TP1
-U 1 1 5E9B5209
-P 4000 2450
-F 0 "TP1" H 3942 2476 50  0000 R CNN
-F 1 "RESET" H 3942 2567 50  0000 R CNN
-F 2 "Connector_PinHeader_2.54mm:PinHeader_1x01_P2.54mm_Vertical" H 4200 2450 50  0001 C CNN
-F 3 "" H 4200 2450 50  0001 C CNN
-	1    4000 2450
-	-1   0    0    1
-$EndComp
 $Comp
 L 4ms-passives:R R2
@@
 F 0 "R2" V 9493 4550 50  0000 C CNN
 F 1 "1k" V 9584 4550 50  0000 C CNN
-F 2 "Resistor_THT:R_Axial_DIN0207_L6.3mm_D2.5mm_P7.62mm_Horizontal" V 9630 4550 50  0001 C CNN
+F 2 "Resistor_THT:R_Axial_DIN0309_L9.0mm_D3.2mm_P2.54mm_Vertical" V 9630 4550 50  0001 C CNN
 F 3 "" H 9700 4550 50  0001 C CNN
 	1    9700 4550
@@
 Wire Wire Line
 	9850 4550 10100 4550
-Text GLabel 3350 6200 2    50   Input ~ 0
-12v
-$Comp
-L 4ms-passives:R R7
-U 1 1 5E0118DA
-P 3250 6500
-F 0 "R7" H 3100 6550 50  0000 C CNN
-F 1 "22k" H 3100 6450 50  0000 C CNN
-F 2 "Resistor_THT:R_Axial_DIN0207_L6.3mm_D2.5mm_P7.62mm_Horizontal" V 3180 6500 50  0001 C CNN
-F 3 "" H 3250 6500 50  0001 C CNN
-	1    3250 6500
-	1    0    0    -1
-$EndComp
+Wire Wire Line
+	2850 6200 2900 6200
+Wire Wire Line
+	3200 6200 3250 6200
+Wire Wire Line
+	3250 6200 3250 6350
+$Comp
+L 4ms-passives:D D3
+U 1 1 5E08C6E3
+P 3050 6200
+F 0 "D3" H 3250 6400 50  0000 C CNN
+F 1 "1N4148" H 3150 6300 50  0000 C CNN
+F 2 "Diode_THT:D_T-1_P5.08mm_Horizontal" H 3050 6200 50  0001 C CNN
+F 3 "" H 3050 6200 50  0001 C CNN
+	1    3050 6200
+	-1   0    0    1
+$EndComp
+Wire Wire Line
+	3250 6650 3250 6750
 $Comp
 L 4ms-power:GND #PWR018
@@
 	1    0    0    -1
 $EndComp
-Wire Wire Line
-	3250 6650 3250 6750
-$Comp
-L 4ms-passives:D D3
-U 1 1 5E08C6E3
-P 3050 6200
-F 0 "D3" H 3250 6400 50  0000 C CNN
-F 1 "1N4148" H 3150 6300 50  0000 C CNN
-F 2 "Diode_THT:D_T-1_P5.08mm_Horizontal" H 3050 6200 50  0001 C CNN
-F 3 "" H 3050 6200 50  0001 C CNN
-	1    3050 6200
-	-1   0    0    1
-$EndComp
-Wire Wire Line
-	3200 6200 3250 6200
-Wire Wire Line
-	3250 6200 3250 6350
+$Comp
+L 4ms-passives:R R7
+U 1 1 5E0118DA
+P 3250 6500
+F 0 "R7" H 3100 6550 50  0000 C CNN
+F 1 "22k" H 3100 6450 50  0000 C CNN
+F 2 "Resistor_THT:R_Axial_DIN0309_L9.0mm_D3.2mm_P2.54mm_Vertical" V 3180 6500 50  0001 C CNN
+F 3 "" H 3250 6500 50  0001 C CNN
+	1    3250 6500
+	1    0    0    -1
+$EndComp
 Connection ~ 3250 6200
 Wire Wire Line
 	3250 6200 3350 6200
-Wire Wire Line
-	2850 6200 2900 6200
+Text GLabel 3350 6200 2    50   Input ~ 0
+12v
+Wire Wire Line
+	1300 3350 2250 3350
+$Comp
+L Mechanical:MountingHole H1
+U 1 1 5E1458CE
+P 9600 5900
+F 0 "H1" H 9700 5946 50  0000 L CNN
+F 1 "MountingHole" H 9700 5855 50  0000 L CNN
+F 2 "MountingHole:MountingHole_3.2mm_M3" H 9600 5900 50  0001 C CNN
+F 3 "~" H 9600 5900 50  0001 C CNN
+	1    9600 5900
+	1    0    0    -1
+$EndComp
+$Comp
+L Mechanical:MountingHole H2
+U 1 1 5E146367
+P 10500 5900
+F 0 "H2" H 10600 5946 50  0000 L CNN
+F 1 "MountingHole" H 10600 5855 50  0000 L CNN
+F 2 "MountingHole:MountingHole_3.2mm_M3" H 10500 5900 50  0001 C CNN
+F 3 "~" H 10500 5900 50  0001 C CNN
+	1    10500 5900
+	1    0    0    -1
+$EndComp
+$Comp
+L Mechanical:MountingHole H3
+U 1 1 5E183F39
+P 9600 6250
+F 0 "H3" H 9700 6296 50  0000 L CNN
+F 1 "MountingHole" H 9700 6205 50  0000 L CNN
+F 2 "MountingHole:MountingHole_3.2mm_M3" H 9600 6250 50  0001 C CNN
+F 3 "~" H 9600 6250 50  0001 C CNN
+	1    9600 6250
+	1    0    0    -1
+$EndComp
+$Comp
+L Mechanical:MountingHole H4
+U 1 1 5E183F43
+P 10500 6250
+F 0 "H4" H 10600 6296 50  0000 L CNN
+F 1 "MountingHole" H 10600 6205 50  0000 L CNN
+F 2 "MountingHole:MountingHole_3.2mm_M3" H 10500 6250 50  0001 C CNN
+F 3 "~" H 10500 6250 50  0001 C CNN
+	1    10500 6250
+	1    0    0    -1
+$EndComp
+Wire Wire Line
+	3900 2350 4100 2350
 $EndSCHEMATC

Commit message: Initial board routings
Connections:
- net TACH1A: now also U1.26 (PC3); no longer U1.24 (PC1)
- net TACH2B: now also U1.3 (PD1); no longer U1.26 (PC3)
- net TACH4A: now also U1.14 (PB0); no longer U1.2 (PD0)
- net TACH4B: now also U1.24 (PC1); no longer U1.3 (PD1)
- net at SW2.2: now also U1.2 (PD0); no longer U1.14 (PB0)
Other:
- moved on the sheet: C2, C3, C4, D3, R1, R7, SW2, U1, X1
